File: integrated_adc.brd (EAGLE design)
At the start: 50.8 x 88.9 mm, 67 parts, among them CON1 UAVCAN_MICRO, CON2 UAVCAN_MICRO, P1 J1B1211CCD, T2 2N7002PS, U1 AP2112K-3.3TRG1, U2 TEENSY_3.X_PINOUT, Y1 NX5032

Commit message: Fix Names and Titles
Parts:
- moved ARVP1 11.7 mm to (17.7, 85.5)
Other:
- board text added: "- David Lenfesty"
- board text added: "- Khang Au - Mohammad Arefin Nazmum"
- board text removed: "David Lenfesty"
- board text removed: "Khang Au Mohammad Arefin"
Changed lines of the file:
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@@
 </layers>
 <board>
-<fusionsync huburn="a.YnVzaW5lc3M6dWFsYmVydGE3NDE" projecturn="a.YnVzaW5lc3M6dWFsYmVydGE3NDEjRDIwMjEwNDE4NDAzOTUxNDI2" f3durn="urn:adsk.wipprod:dm.lineage:qySGYL3aS7Sd287As8-wjA" pcbguid="" lastpulledtime="" lastsyncedchangeguid="" latestrevisionid="7eceeb94-81c8-46be-9b74-f53db65ab365" lastsyncedrevisionid="7eceeb94-81c8-46be-9b74-f53db65ab365" lastboardhashguid="1e44af1c-a660-02b3-6b96-4401e9e21ad5" lastpushedtime="2021-08-14T18:28:27Z" linktopcb3d="false"/>
+<fusionsync huburn="a.YnVzaW5lc3M6dWFsYmVydGE3NDE" projecturn="a.YnVzaW5lc3M6dWFsYmVydGE3NDEjRDIwMjEwNDE4NDAzOTUxNDI2" f3durn="urn:adsk.wipprod:dm.lineage:qySGYL3aS7Sd287As8-wjA" pcbguid="" lastpulledtime="" lastsyncedchangeguid="" latestrevisionid="7eceeb94-81c8-46be-9b74-f53db65ab365" lastsyncedrevisionid="7eceeb94-81c8-46be-9b74-f53db65ab365" lastboardhashguid="1e44af1c-a660-02b3-6b96-4401e9e21ad5" lastpushedtime="2021-08-14T18:28:27Z" linktopcb3d="true"/>
 <plain>
 <wire x1="0" y1="1.27" x2="0" y2="87.63" width="0.1524" layer="20"/>
@@
 <text x="17.907" y="54.737" size="0.762" layer="21" rot="R90" align="bottom-right">DTR</text>
 <text x="39.4208" y="57.0484" size="1.016" layer="21" rot="R90" align="bottom-right">CAN</text>
-<text x="43.1038" y="84.2264" size="1.27" layer="21" rot="SR0" align="bottom-right">Sonar Data Acquisition Board</text>
+<text x="38.2524" y="83.2104" size="1.524" layer="21" rot="SR0" align="bottom-right">Sonar Data Acquisition Board</text>
 <text x="32.258" y="1.651" size="1.016" layer="21" rot="R90">Reset</text>
 <text x="36.83" y="2.921" size="1.016" layer="21">Boot Select</text>
@@
 <hole x="46.99" y="83.82" drill="3.5"/>
 <hole x="3.81" y="83.82" drill="3.5"/>
-<text x="29.3624" y="86.7156" size="1.524" layer="21">David Lenfesty</text>
+<text x="32.6136" y="78.3844" size="1.4224" layer="21">- David Lenfesty</text>
 <wire x1="49.53" y1="0" x2="1.27" y2="0" width="0.1524" layer="20"/>
 <wire x1="49.53" y1="88.9" x2="50.8" y2="87.63" width="0.1524" layer="20" curve="-90"/>
@@
 <wire x1="1.27" y1="0" x2="0" y2="1.27" width="0.1524" layer="20" curve="-90"/>
 <wire x1="50.8" y1="1.27" x2="49.53" y2="0" width="0.1524" layer="20" curve="-90"/>
-<text x="45.4152" y="83.6168" size="1.4224" layer="21" rot="R180">Khang Au
-Mohammad Arefin</text>
+<text x="50.1396" y="77.724" size="1.4224" layer="21" rot="R180">- Khang Au
+- Mohammad Arefin
+  Nazmum</text>
 </plain>
 <attributes>
@@
 <element name="U$3" library="integrated_adc" package="LQFP100" value="STM32F303VE" x="20.32" y="26.67" smashed="yes" rot="R270">
 <attribute name="NAME" x="28.94" y="32.845" size="1.27" layer="25" rot="R270"/>
-<attribute name="VALUE" x="19.225" y="31.805" size="1.27" layer="27" rot="R270"/>
+<attribute name="VALUE" x="14.4738" y="28.0642" size="1.27" layer="27"/>
 </element>
 <element name="U$4" library="integrated_adc" package="AMPHENOL_MICROB_SMD" value="AMPHENOL_MICROB-USB" x="1.9304" y="53.3908" smashed="yes" rot="R270"/>
@@
 <attribute name="VALUE" x="35.4838" y="43.8404" size="1.27" layer="27"/>
 </element>
-<element name="ARVP1" library="ARVP" package="ARVP" value="ARVP_LOGO" x="5.969" y="85.471" smashed="yes"/>
+<element name="ARVP1" library="ARVP" package="ARVP" value="ARVP_LOGO" x="17.7038" y="85.5472" smashed="yes"/>
 <element name="JP4" library="pinhead" library_urn="urn:adsk.eagle:library:325" package="1X03" package3d_urn="urn:adsk.eagle:package:22458/2" value="" x="40.513" y="6.223" smashed="yes">
 <attribute name="VALUE" x="36.703" y="3.048" size="1.27" layer="27"/>
@@
 <wire x1="22.3774" y1="63.754" x2="23.2156" y2="63.754" width="0.3048" layer="1"/>
 <wire x1="23.2156" y1="63.754" x2="23.4696" y2="64.008" width="0.3048" layer="1"/>
-<wire x1="27.597146875" y1="53.682853125" x2="26.8328" y2="52.91850625" width="0.3048" layer="1"/>
+<wire x1="27.7746" y1="53.86030625" x2="26.8328" y2="52.91850625" width="0.3048" layer="1"/>
 <wire x1="44.9208" y1="56.485" x2="44.45" y2="56.9558" width="0.2032" layer="1"/>
 <contactref element="P1" pad="9"/>
@@
 <via x="13.081" y="58.4454" extent="1-16" drill="0.35"/>
 <wire x1="27.7746" y1="54.401" x2="27.7746" y2="53.86030625" width="0.3048" layer="1"/>
-<wire x1="27.7746" y1="53.86030625" x2="27.597146875" y2="53.682853125" width="0.3048" layer="1"/>
 </signal>
 <signal name="!RST">
@@
 <wire x1="36.703" y1="20.32" x2="36.703" y2="23.368" width="0.2032" layer="1"/>
 <wire x1="36.703" y1="23.368" x2="37.395" y2="24.06" width="0.2032" layer="1"/>
-<wire x1="37.395" y1="24.06" x2="38.1" y2="24.06" width="0.2032" layer="1"/>
-<wire x1="38.1" y1="24.06" x2="38.227" y2="24.06" width="0.2032" layer="1"/>
+<wire x1="37.395" y1="24.06" x2="38.227" y2="24.06" width="0.2032" layer="1"/>
 <wire x1="30.0962" y1="17.0152" x2="32.131" y2="19.05" width="0.2032" layer="1"/>
 <contactref element="R4" pad="1"/>
 <wire x1="37.465" y1="29.149" x2="37.465" y2="26.416" width="0.254" layer="1"/>
-<wire x1="38.227" y1="25.654" x2="38.227" y2="24.003" width="0.254" layer="1"/>
+<wire x1="38.227" y1="25.654" x2="38.227" y2="24.06" width="0.254" layer="1"/>
 <wire x1="38.227" y1="24.06" x2="38.227" y2="24.003" width="0.254" layer="1"/>
 <wire x1="37.465" y1="26.416" x2="38.227" y2="25.654" width="0.254" layer="1"/>
